File: Kicad_porting/diyscip-v2.sch (KiCad schematic (older format))
At the start: 30 parts, among them IC1 CD4051BE, IC2 CD4051BE, IC3 SN74HC595N, IC4 SN74HC595N, J1 Conn_01x05_Male, J3 Conn_01x05_Male, Q1 BSS138, Q2 BSS138, Q3 BSS138, U1 AMS1117-3.3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

Commit message: Aggiunta resistenza "dimenticata" su segnale DATA
Parts:
- added R15: 1K, Resistor_SMD:R_0603_1608Metric, symbol Device:R
Connections:
- wire segments 247 -> 253
Changed lines of the file:
@@
 	7750 1500 7950 1500
 Wire Wire Line
-	7950 1500 7950 3200
+	7950 1500 7950 2400
 Wire Wire Line
 	7950 3200 7750 3200
@@
 Wire Wire Line
 	10550 1400 10800 1400
-Wire Wire Line
-	9700 1500 10550 1500
 $Comp
 L power:GND #PWR017
@@
 Wire Wire Line
 	9850 1600 9850 2200
-Wire Wire Line
-	9850 2200 8550 2200
 Wire Wire Line
 	8550 2200 8550 2250
@@
 Text Notes 3500 4250 0    50   ~ 0
 Signal\nconversion\n5v —> 3.3v
+$Comp
+L Device:R R15
+U 1 1 60046BE8
+P 10200 2300
+F 0 "R15" V 9993 2300 50  0000 C CNN
+F 1 "1K" V 10084 2300 50  0000 C CNN
+F 2 "Resistor_SMD:R_0603_1608Metric" V 10130 2300 50  0001 C CNN
+F 3 "~" H 10200 2300 50  0001 C CNN
+F 4 "C21190" H 10200 2300 50  0001 C CNN "LCSC"
+	1    10200 2300
+	0    1    1    0
+$EndComp
+Wire Wire Line
+	10350 2300 10350 1500
+Wire Wire Line
+	9700 1500 10350 1500
+Connection ~ 10350 1500
+Wire Wire Line
+	10350 1500 10550 1500
+Wire Wire Line
+	8550 2200 9850 2200
+Wire Wire Line
+	10050 2300 9100 2300
+Wire Wire Line
+	9100 2300 9100 2400
+Wire Wire Line
+	9100 2400 7950 2400
+Connection ~ 7950 2400
+Wire Wire Line
+	7950 2400 7950 3200
 $EndSCHEMATC
